Commit message: Add H1-2 wrist control dashboard

File: static/models/h1_2_description/h1_2.urdf (robot description, URDF)
Before this commit: robot h1_2, 58 links, 57 joints
Joints:
- joint R_base_link_joint: origin xyz=0.054 0 0 rpy=3.1415926535897932384626433832795 0 -1.5707963267948966192313216916398 -> xyz=0.054 0 0 rpy=3.1415926535897932384626433832795 0 1.5707963267948966192313216916398
